File: hardware/teensy_4p0_shield/TeensyKeyerShield.kicad_pcb (KiCad board)
At the start: 2 copper layers, 100 x 50 mm, 99 parts, among them J1 Conn_01x02, J10 Conn_01x04, J11 Conn_02x05_Odd_Even, J12 AudioJack3_SwitchTR, J2 Conn_01x02, J3 Conn_01x02, J4 Conn_01x02, J5 AudioJack3_SwitchTR, J6 AudioJack3_SwitchTR, J7 AudioJack3_SwitchTR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

Commit message: 0p91 shield release
Connections:
- MIC1 pad 1: Net-(C24-Pad1) -> Net-(C25-Pad1)
- MIC1 pad 4: Net-(C25-Pad1) -> Net-(C24-Pad1)
Routing:
- net Net-(C25-Pad1): track 3.50 -> 5.95 mm
Other:
- board text added: "CW Keyer Shield 0.91 © 2021 SofterHardware"
- board text removed: "CW Keyer Shield 0.9 © 2021 SofterHardware"
Changed lines of the file:
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@@
-(kicad_pcb (version 20171130) (host pcbnew 5.1.11-e4df9d881f~92~ubuntu20.04.1)
+(kicad_pcb (version 20171130) (host pcbnew 5.1.12-84ad8e8a86~92~ubuntu20.04.1)
   (general
     (thickness 1.6)
     (drawings 50)
-    (tracks 838)
+    (tracks 839)
     (zones 0)
     (modules 99)
@@
   (title_block
     (title "CW Keyer Shield")
-    (date 2021-11-07)
+    (date 2021-11-09)
+    (rev 0.91)
     (company Softerhardware)
     (comment 1 "KF7O Steve Haynal")
@@
     (fp_arc (start 2.4 -0.7) (end 2.4 -0.5) (angle -270) (layer F.SilkS) (width 0.12))
     (pad 4 smd circle (at 0 0 90) (size 0.9 0.9) (layers F.Cu F.Paste F.Mask)
-      (net 24 "Net-(C25-Pad1)"))
+      (net 23 "Net-(C24-Pad1)"))
     (pad 3 smd circle (at 0 2.46 90) (size 0.9 0.9) (layers F.Cu F.Paste F.Mask)
       (net 2 GND))
@@
       (net 2 GND))
     (pad 1 smd circle (at 1.7 0 90) (size 0.9 0.9) (layers F.Cu F.Paste F.Mask)
-      (net 23 "Net-(C24-Pad1)"))
+      (net 24 "Net-(C25-Pad1)"))
   )
   (module Resistor_SMD:R_0603_1608Metric_Pad0.98x0.95mm_HandSolder (layer F.Cu)
@@
     (effects (font (size 1 1) (thickness 0.15)))
   )
-  (gr_text "CW Keyer Shield 0.9\n© 2021 SofterHardware" (at 96.1 73.1) (layer F.SilkS)
+  (gr_text "CW Keyer Shield 0.91\n© 2021 SofterHardware" (at 96.1 73.1) (layer F.SilkS)
     (effects (font (size 1 1) (thickness 0.15)) (justify left))
   )
@@
   (segment (start 114.1 106.75) (end 114.15 106.7) (width 0.25) (layer F.Cu) (net 23))
   (segment (start 114.1 108.3) (end 114.1 106.75) (width 0.25) (layer F.Cu) (net 23))
-  (segment (start 114.25 106.6) (end 114.15 106.7) (width 0.25) (layer F.Cu) (net 23))
-  (segment (start 116 106.6) (end 114.25 106.6) (width 0.25) (layer F.Cu) (net 23))
+  (segment (start 116 108.3) (end 114.1 108.3) (width 0.25) (layer F.Cu) (net 23))
   (segment (start 114.1 109.9) (end 116 109.9) (width 0.25) (layer F.Cu) (net 24))
-  (segment (start 116 108.3) (end 116 109.9) (width 0.25) (layer F.Cu) (net 24))
+  (segment (start 116.9 107.5) (end 116 106.6) (width 0.25) (layer F.Cu) (net 24))
+  (segment (start 116.9 109) (end 116.9 107.5) (width 0.25) (layer F.Cu) (net 24))
+  (segment (start 116 109.9) (end 116.9 109) (width 0.25) (layer F.Cu) (net 24))
   (segment (start 110.325 112.7) (end 110.5 112.525) (width 0.25) (layer F.Cu) (net 25))
   (segment (start 100.5 118) (end 100.5 115.7) (width 0.25) (layer F.Cu) (net 25))
